File: big_muff_pi.kicad_sch (KiCad schematic)
At the start: 70 parts, among them J1 NMJ6HHD2, J2 NMJ6HHD2, J3 Conn_01x05, J4 Conn_01x05, J5 Conn_01x05, J6 Barrel_Jack_MountingPin, Q1 MMBT5551, Q2 MMBT5551, Q3 MMBT5551, Q4 MMBT5551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

Commit message: Estetics finalized.
Parts:
- removed RV1, RV2, RV3: 100k, Potentiometer_THT:Potentiometer_Alpha_RD901F-40-00D_Single_Vertical, symbol Device:R_Potentiometer
- added D8: floating_green_led, pedale:floating_green_led, symbol pedale:floating_green_led
- added D9: floating_red_led, pedale:floating_red_led, symbol pedale:floating_red_led
- added H5: MountingHole, pedale:M3_hole_with_spacer, symbol Mechanical:MountingHole
- added RV1, RV2, RV3: floating_pot_knob, pedale:floating_pot_knob, symbol pedale:floating_pot_knob
- added RV4, RV5, RV6: floating_pot, pedale:floating_pot, symbol pedale:floating_pot
Other:
- moved on the sheet: H1, H2, H3, H4

Commit message: Est
Parts:
- removed D6: LED, LED_THT:LED_D5.0mm, symbol Device:LED
- removed R23: 1k, Resistor_SMD:R_0603_1608Metric_Pad0.98x0.95mm_HandSolder, symbol Device:R
- added P1: big_muff_pi_front_panel, pedale:big_muff_pi_front_plate, symbol pedale:big_muff_pi_front_panel
- added R25, R26: 1k, Resistor_SMD:R_0603_1608Metric_Pad0.98x0.95mm_HandSolder, symbol Device:R
- added SIM1: Logo_Open_Hardware_Small, Symbol:OSHW-Logo2_7.3x6mm_SilkScreen, symbol Graphic:Logo_Open_Hardware_Small
Connections:
- net 0: now also R25.2, R26.2; no longer J3.1 (Pin_1), J3.5 (Pin_5), J5.1 (Pin_1), J5.5 (Pin_5)
- net 9V: now also J3.1 (Pin_1)
- net FS_OUT: now also J3.4 (Pin_4); no longer J3.2 (Pin_2)
- net at R6.1: now also J3.2 (Pin_2); no longer J3.4 (Pin_4)
- net at SW1.5 (B): now also J5.5 (Pin_5)
- new net: J3.5 (Pin_5), R25.1
- new net: J5.1 (Pin_1), R26.1
- no-connect marks 2 -> 3
Other:
- moved on the sheet: D8, D9, J3, R6, RV1, RV3, RV4, RV6, SW1B

Commit message: Only routing left.
Connections:
- net 0: now also J1.S, J2.S, J4.4 (Pin_4), J5.1 (Pin_1); no longer J4.1 (Pin_1), J5.2 (Pin_2)
- net 9V: now also J3.4 (Pin_4); no longer J3.1 (Pin_1)
- net FS_OUT: now also J3.3 (Pin_3); no longer J3.4 (Pin_4)
- net F_OUT: now also J4.2 (Pin_2); no longer J4.3 (Pin_3)
- net at R6.1: now also J3.1 (Pin_1); no longer J3.2 (Pin_2)
- net at R7.1: now also J3.2 (Pin_2); no longer J3.3 (Pin_3)
- net at R26.1: now also J5.5 (Pin_5); no longer J5.1 (Pin_1)
- net at C12.2, R22.2: now also J4.3 (Pin_3); no longer J4.4 (Pin_4)
- net at C13.2, R17.2: now also J4.1 (Pin_1); no longer J4.2 (Pin_2)
- net at SW1.1 (A): now also J5.2 (Pin_2); no longer J5.3 (Pin_3)
- net at SW1.5 (B): now also J5.4 (Pin_4); no longer J5.5 (Pin_5)
- net at C11.2: now also J5.3 (Pin_3); no longer J5.4 (Pin_4)
- no-connect marks 3 -> 2
Other:
- note added: "Clipping and tone stage"
- note added: "Input gain stage"
- note added: "Mounting and estetics"
- note added: "Output gain stage and selection switch"
- note added: "Power supply"
- note removed: "DODATI 3D PRINTED PLASTIKU ISPOD PCB-A"
- note removed: "NAPRAVI FACE PLATE PCB"
- note removed: "Rupe za montiranje"
- note removed: "SELEKTUJ DEBLJI PCB"
- title: (none) -> Big Muff Pi
- moved on the sheet: BT1, C1, C10, C11, C12, C13, C14, C16, C17, C18, C19, C2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
