File: big_muff_pi.kicad_pcb (KiCad board)
At the start: 2 copper layers, 80 x 100 mm, 78 parts, among them J1 NMJ6HHD2, J2 NMJ6HHD2, J3 Conn_01x05, J4 Conn_01x05, J5 Conn_01x05, J6 Barrel_Jack_MountingPin, P1 big_muff_pi_front_panel, Q1 MMBT5551, Q2 MMBT5551, Q3 MMBT5551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

Commit message: poredjane komponente
Parts:
- moved R5 19.9 mm to (54.5, 61.4), turned to 0 degrees
- moved C10 18.7 mm to (100.6, 59.1), turned to -90 degrees
- moved R4 16.4 mm to (53.9, 64.0), turned to 90 degrees
- moved C1 14.7 mm to (55.6, 64.0), turned to 90 degrees
- moved C3 13.3 mm to (61.0, 62.3), turned to 90 degrees
- moved Q4 12.5 mm to (58.2, 64.1), turned to 90 degrees
- moved R1 10.9 mm to (56.0, 68.1), turned to -90 degrees
- moved R17 10.7 mm to (90.6, 64.9), turned to 180 degrees
- moved R20 10.3 mm to (103.6, 66.2)
- moved C11 10.2 mm to (103.6, 62.7)
- moved R19 10.1 mm to (100.6, 61.7)
- moved Q3 9.95 mm to (100.7, 66.1)
- moved R21 9.95 mm to (100.5, 68.7)
- moved C13 9.95 mm to (87.0, 64.8), turned to 0 degrees
- moved R18 9.93 mm to (100.6, 63.5)
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
Commit message: rutiranje v1
Parts:
- moved R6 17.7 mm to (62.1, 59.1), turned to 180 degrees
- moved R2 16.6 mm to (78.4, 64.9)
- moved C1 16.6 mm to (72.2, 63.7)
- moved R3 16.6 mm to (77.0, 68.7)
- moved R4 16.6 mm to (70.5, 63.7)
- moved C2 16.6 mm to (74.3, 67.8)
- moved Q4 16.6 mm to (74.8, 63.8)
- moved R1 16.6 mm to (72.6, 67.8)
- moved R5 16.6 mm to (71.1, 61.1)
- moved R20 11.1 mm to (114.6, 67.3)
- moved C11 11.0 mm to (114.6, 63.4)
- moved C3 10.5 mm to (71.1, 59.5), turned to 180 degrees
- moved C10 8.86 mm to (109.4, 60.1)
- moved R18 8.86 mm to (109.4, 64.5)
- moved Q3 8.86 mm to (109.5, 67.1)
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Routing:
- net 9V: track 0.00 -> 212.6 mm, vias 0 -> 3
- net Net-(J5-Pin_4): track 0.00 -> 100.2 mm
- net Net-(J5-Pin_2): track 0.00 -> 79.6 mm, vias 0 -> 4
- net SW_IN: track 0.00 -> 78.0 mm, vias 0 -> 4
- net Net-(SW1A-B): track 0.00 -> 30.4 mm
- net F_OUT: track 0.00 -> 29.5 mm
- net Net-(D1-A): track 0.00 -> 22.3 mm
- net Net-(J3-Pin_2): track 0.00 -> 19.4 mm
- net Net-(Q2-B): track 0.00 -> 18.9 mm
- net 0: track 0.00 -> 18.9 mm, vias 0 -> 17
- net Net-(D4-K): track 0.00 -> 17.3 mm
- net Net-(D3-K): track 0.00 -> 17.0 mm
- net Net-(J4-Pin_3): track 0.00 -> 13.8 mm
- net Net-(J4-Pin_1): track 0.00 -> 12.9 mm
- net Net-(Q1-B): track 0.00 -> 12.1 mm
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
Commit message: rutiranje v2.
Routing:
- net 9V: track 212.6 -> 227.4 mm
- net Net-(Q4-C): track 10.6 -> 7.65 mm
- net F_OUT: track 29.5 -> 28.0 mm
- net Net-(J5-Pin_4): track 100.2 -> 98.9 mm
- net Net-(J5-Pin_2): track 79.6 -> 80.1 mm
