File: big_muff_pi.kicad_pcb (KiCad board)
At the start: 2 copper layers, 80 x 100 mm, 78 parts, among them J1 NMJ6HHD2, J2 NMJ6HHD2, J3 Conn_01x05, J4 Conn_01x05, J5 Conn_01x05, J6 Barrel_Jack_MountingPin, P1 big_muff_pi_front_panel, Q1 MMBT5551, Q2 MMBT5551, Q3 MMBT5551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

Commit message: Tiny changes.
Routing:
- net Net-(Q5-B): track 11.7 -> 12.4 mm
- net 0: vias 17 -> 64
- added copper zone on F.Cu, net 0

Commit message: Updated library.
Parts:
- removed J6: Barrel_Jack_MountingPin, Connector_BarrelJack:BarrelJack_GCT_DCJ200-10-A_Horizontal
- removed RV1, RV2, RV3: floating_pot_knob, pedale:floating_pot_knob
- added J7: Conn_01x01_Socket, TestPoint:TestPoint_THTPad_D2.5mm_Drill1.2mm, F.Cu at (69.0, 89.6)
- added J8: Conn_01x01_Socket, TestPoint:TestPoint_THTPad_D2.5mm_Drill1.2mm, F.Cu at (68.9, 102.4)
- added J9: Barrel_Jack_Switch, pedale:BarrelJack, F.Cu at (63.9, 103.3)
- J1, J2: value NMJ6HHD2 -> Jack_6.35; footprint Connector_Audio:Jack_6.35mm_Neutrik_NMJ6HHD2_Horizontal -> pedale:Jack_6.35mm
- SW1: footprint pedale:foot_switch -> pedale:foot_switch_tht_and_floating
- moved SW1 9.30 mm to (90.0, 125.0)
- moved BT1 4.15 mm to (75.0, 89.7)
Connections:
- BT1 pad 2: 0 -> Net-(BT1--)
Routing:
- net Net-(BT1--): track 0.00 -> 17.5 mm
- net 9V: track 227.4 -> 220.5 mm, vias 3 -> 5
- net Net-(BT1-+): track 9.61 -> 15.5 mm
- net Net-(J5-Pin_4): track 98.9 -> 93.2 mm, vias 0 -> 2
- net Net-(Q5-B): track 12.4 -> 11.2 mm
- net Net-(SW1A-B): track 30.4 -> 31.2 mm
- net 0: vias 64 -> 62
