File: big_muff_pi.kicad_pcb (KiCad board)
At the start: 2 copper layers, 80 x 100 mm, 77 parts, among them J1 Jack_6.35, J2 Jack_6.35, J3 Conn_01x05, J4 Conn_01x05, J5 Conn_01x05, J7 Conn_01x01_Socket, J8 Conn_01x01_Socket, J9 Barrel_Jack_Switch, P1 big_muff_pi_front_panel, Q1 MMBT5551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

Commit message: Rotated 6.35 pins, switched connector positions, switched LED.
Parts:
- moved J1 48.4 mm to (67.2, 133.1), turned to 180 degrees
- moved J2 48.4 mm to (112.8, 116.9), turned to 0 degrees
Connections:
- SW1 pad 1: Net-(J5-Pin_2) -> SW_IN
- SW1 pad 3: SW_IN -> Net-(J5-Pin_2)
Routing:
- net Net-(J5-Pin_2): track 80.1 -> 70.5 mm
- net Net-(J5-Pin_4): track 93.2 -> 100.1 mm
- net SW_IN: track 78.0 -> 82.7 mm
- net Net-(SW1A-B): track 31.2 -> 29.4 mm
- net 0: vias 62 -> 60
