File: big_muff_pi/big_muff_pi.kicad_sch (KiCad schematic)
At the start: 81 parts, among them J1 Jack_6.35, J2 Jack_6.35, J6 top_panel_connector, J7 Conn_01x01_Socket, J8 Conn_01x01_Socket, J9 Barrel_Jack_Switch, P1 big_muff_pi_front_panel, Q1 MMBT5551, Q10 AO3401A, Q12 AO3400A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

Commit message: small work
Parts:
- added P2: bottom_panel, pedale:bottom_plate, symbol pedale:big_muff_pi_front_panel
Changed lines of the file:
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@@
+	)
+	(symbol
+		(lib_id "pedale:big_muff_pi_front_panel")
+		(at 76.2 90.17 0)
+		(unit 1)
+		(exclude_from_sim no)
+		(in_bom yes)
+		(on_board yes)
+		(dnp no)
+		(fields_autoplaced yes)
+		(property "Reference" "P2"
+			(at 78.74 88.8999 0)
+			(effects
+				(font
+					(size 1.27 1.27)
+				)
+				(justify left)
+			)
+		)
+		(property "Value" "bottom_panel"
+			(at 78.74 91.4399 0)
+			(effects
+				(font
+					(size 1.27 1.27)
+				)
+				(justify left)
+			)
+		)
+		(property "Footprint" "pedale:bottom_plate"
+			(at 76.2 90.17 0)
+			(effects
+				(font
+					(size 1.27 1.27)
+				)
+				(hide yes)
+			)
+		)
+		(property "Datasheet" "~"
+			(at 76.2 90.17 0)
+			(effects
+				(font
+					(size 1.27 1.27)
+				)
+				(hide yes)
+			)
+		)
+		(property "Description" "Potentiometer"
+			(at 76.2 90.17 0)
+			(effects
+				(font
+					(size 1.27 1.27)
+				)
+				(hide yes)
+			)
+		)
+		(instances
+			(project "big_muff_pi"
+				(path "/1fda0e48-ac05-4486-b24b-352a2425b266"
+					(reference "P2")
+					(unit 1)
+				)
+			)
+		)
 	)
 	(symbol

Commit message: small.
Parts:
- removed D8: floating_green_led, pedale:floating_green_led, symbol pedale:floating_green_led
- removed D9: floating_red_led, pedale:floating_red_led, symbol pedale:floating_red_led
- removed RV4, RV5, RV6: floating_pot, pedale:floating_pot, symbol pedale:floating_pot
- P1: value big_muff_pi_front_panel -> front_panel; footprint pedale:big_muff_pi_front_plate -> pedale:front_plate
Connections:
- net 0: no longer J1.R, J2.R
- no-connect marks 1 -> 4
Other:
- note added: "Power supply filtering"
- note removed: "Mounting and estetics"
- moved on the sheet: H1, H2, H3, H4, H5, P1, P2
