File: big_muff_pi_front_plate/big_muff_pi_front_plate.kicad_pcb (KiCad board)
At the start: 2 copper layers, 80 x 100 mm, 12 parts, among them J1 top_panel_connector

Commit message: Pot labels.
Other:
- board text added: "100 kOhm lin"
Changed lines of the file:
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@@
+		)
+	)
+	(gr_text "100 kOhm lin"
+		(at 94.9 89.8 0)
+		(layer "B.SilkS")
+		(effects
+			(font
+				(size 1 1)
+				(thickness 0.15)
+			)
+			(justify left bottom mirror)
+		)
+	)
+	(gr_text "100 kOhm lin"
+		(at 116.9 79.5 0)
+		(layer "B.SilkS")
+		(effects
+			(font
+				(size 1 1)
+				(thickness 0.15)
+			)
+			(justify left bottom mirror)
+		)
+	)
+	(gr_text "100 kOhm lin"
+		(at 73.1 79.5 0)
+		(layer "B.SilkS")
+		(effects
+			(font
+				(size 1 1)
+				(thickness 0.15)
+			)
+			(justify left bottom mirror)
 		)
 	)

Commit message: dfasdf dfasdf
Changed lines of the file:
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@@
-		)
-		(fp_line
-			(start -4.68 0.5)
-			(end -4.68 -0.5)
-			(stroke
-				(width 0.12)
-				(type solid)
-			)
-			(layer "B.SilkS")
-		)
-		(fp_line
-			(start -3.68 0)
-			(end -4.68 0.5)
-			(stroke
-				(width 0.12)
-				(type solid)
-			)
-			(layer "B.SilkS")
-		)
-		(fp_line
-			(start -4.68 -0.5)
-			(end -3.68 0)
-			(stroke
-				(width 0.12)
-				(type solid)
-			)
-			(layer "B.SilkS")
 		)
 		(fp_line
@@
 		(pad "1" smd roundrect
 			(at -0.2 0 270)
-			(size 3.31 1.7)
+			(size 3.31 1.2)
 			(drill
 				(offset -0.575 0)
@@
 		(pad "2" smd roundrect
 			(at 3.345 0 270)
-			(size 3.31 1.7)
+			(size 3.31 1.2)
 			(layers "B.Cu" "B.Mask")
 			(roundrect_rratio 0.1470588235)
@@
 		(pad "3" smd roundrect
 			(at -0.775 -2.54 270)
-			(size 3.31 1.7)
+			(size 3.31 1.2)
 			(layers "B.Cu" "B.Mask")
 			(roundrect_rratio 0.1470588235)
@@
 		(pad "4" smd roundrect
 			(at 3.345 -2.54 270)
-			(size 3.31 1.7)
+			(size 3.31 1.2)
 			(layers "B.Cu" "B.Mask")
 			(roundrect_rratio 0.1470588235)
@@
 		(pad "5" smd roundrect
 			(at -0.775 -5.08 270)
-			(size 3.31 1.7)
+			(size 3.31 1.2)
 			(layers "B.Cu" "B.Mask")
 			(roundrect_rratio 0.1470588235)
@@
 		(pad "6" smd roundrect
 			(at 3.345 -5.08 270)
-			(size 3.31 1.7)
+			(size 3.31 1.2)
 			(layers "B.Cu" "B.Mask")
 			(roundrect_rratio 0.1470588235)
@@
 		(pad "7" smd roundrect
 			(at -0.775 -7.62 270)
-			(size 3.31 1.7)
+			(size 3.31 1.2)
 			(layers "B.Cu" "B.Mask")
 			(roundrect_rratio 0.1470588235)
@@
 		(pad "8" smd roundrect
 			(at 3.345 -7.62 270)
-			(size 3.31 1.7)
+			(size 3.31 1.2)
 			(layers "B.Cu" "B.Mask")
 			(roundrect_rratio 0.1470588235)
@@
 		(pad "9" smd roundrect
 			(at -0.775 -10.16 270)
-			(size 3.31 1.7)
+			(size 3.31 1.2)
 			(layers "B.Cu" "B.Mask")
 			(roundrect_rratio 0.1470588235)
@@
 		(pad "10" smd roundrect
 			(at 3.345 -10.16 270)
-			(size 3.31 1.7)
+			(size 3.31 1.2)
 			(layers "B.Cu" "B.Mask")
 			(roundrect_rratio 0.1470588235)
@@
 		(pad "11" smd roundrect
 			(at -0.775 -12.7 270)
-			(size 3.31 1.7)
+			(size 3.31 1.2)
 			(layers "B.Cu" "B.Mask")
 			(roundrect_rratio 0.1470588235)
@@
 		(pad "12" smd roundrect
 			(at 3.345 -12.7 270)
-			(size 3.31 1.7)
+			(size 3.31 1.2)
 			(layers "B.Cu" "B.Mask")
 			(roundrect_rratio 0.1470588235)
@@
 		(pad "13" smd roundrect
 			(at -0.775 -15.24 270)
-			(size 3.31 1.7)
+			(size 3.31 1.2)
 			(layers "B.Cu" "B.Mask")
 			(roundrect_rratio 0.1470588235)
@@
 		(pad "14" smd roundrect
 			(at 3.345 -15.24 270)
-			(size 3.31 1.7)
+			(size 3.31 1.2)
 			(layers "B.Cu" "B.Mask")
 			(roundrect_rratio 0.1470588235)
@@
 		(pad "15" smd roundrect
 			(at -0.775 -17.78 270)
-			(size 3.31 1.7)
+			(size 3.31 1.2)
 			(layers "B.Cu" "B.Mask")
 			(roundrect_rratio 0.1470588235)
@@
 		(pad "16" smd roundrect
 			(at 3.345 -17.78 270)
-			(size 3.31 1.7)
+			(size 3.31 1.2)
 			(layers "B.Cu" "B.Mask")
 			(roundrect_rratio 0.1470588235)
@@
 		)
 		(embedded_fonts no)
-		(model "${KICAD9_3DMODEL_DIR}/Connector_IDC.3dshapes/IDC-Header_2x08_P2.54mm_Vertical.wrl"
+		(model "${KIPRJMOD}/../pedale.pretty/IDC-Header_2x08_P2.54mm_Vertical.stp"
 			(offset
 				(xyz 0 0 3)
@@
 			)
 			(rotate
-				(xyz -0 -0 -0)
-			)
-		)
+				(xyz -0 -0 90)
+			)
+		)
+		(model "${KIPRJMOD}/../pedale.pretty/IDC_female_16_no_strain.step"
+			(offset
+				(xyz 1.5 -8.9 12)
+			)
+			(scale
+				(xyz 1 1 1)
+			)
+			(rotate
+				(xyz -90 -0 -90)
+			)
+		)
